File: PWMGenerator-nkoirala1/PWMGenerator-nkoirala1.kicad_sch (KiCad schematic)
At the start: 0 parts

Commit message: COmmit
Parts:
- added D1: LED, symbol Device:LED
- added J1: Barrel_Jack, symbol Connector:Barrel_Jack
- added Q1: NPN, symbol Simulation_SPICE:NPN
- added Q2: PNP, symbol Simulation_SPICE:PNP
- added RV1: R_Potentiometer, symbol Device:R_Potentiometer
- added U1, U2: LM7805_TO220, Package_TO_SOT_THT:TO-220-3_Vertical, symbol Regulator_Linear:LM7805_TO220

Commit message: Added Commponent
Parts:
- removed U2: LM7805_TO220, Package_TO_SOT_THT:TO-220-3_Vertical, symbol Regulator_Linear:LM7805_TO220
- added J2: Conn_01x03_Pin, Connector_PinHeader_2.54mm:PinHeader_1x03_P2.54mm_Vertical, symbol Connector:Conn_01x03_Pin
- D1: footprint (none) -> LED_THT:LED_D5.0mm
- J1: footprint (none) -> Connector_BarrelJack:BarrelJack_CLIFF_FC681465S_SMT_Horizontal
- Q1, Q2: footprint (none) -> Package_TO_SOT_THT:TO-92
- RV1: footprint (none) -> Potentiometer_THT:Potentiometer_Bourns_3296W_Vertical
Changed lines of the file:
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@@
-	)
-	(symbol
-		(lib_id "Regulator_Linear:LM7805_TO220")
-		(at 779.78 83.82 0)
-		(unit 1)
-		(exclude_from_sim no)
-		(in_bom yes)
-		(on_board yes)
-		(dnp no)
-		(fields_autoplaced yes)
-		(property "Reference" "U2"
-			(at 779.78 77.47 0)
-			(effects
-				(font
-					(size 1.27 1.27)
-				)
-			)
-		)
-		(property "Value" "LM7805_TO220"
-			(at 779.78 80.01 0)
-			(effects
-				(font
-					(size 1.27 1.27)
-				)
-			)
-		)
-		(property "Footprint" "Package_TO_SOT_THT:TO-220-3_Vertical"
-			(at 779.78 78.105 0)
-			(effects
-				(font
-					(size 1.27 1.27)
-					(italic yes)
-				)
-				(hide yes)
-			)
-		)
-		(property "Datasheet" "https://www.onsemi.cn/PowerSolutions/document/MC7800-D.PDF"
-			(at 779.78 85.09 0)
-			(effects
-				(font
-					(size 1.27 1.27)
-				)
-				(hide yes)
-			)
-		)
-		(property "Description" "Positive 1A 35V Linear Regulator, Fixed Output 5V, TO-220"
-			(at 779.78 83.82 0)
-			(effects
-				(font
-					(size 1.27 1.27)
-				)
-				(hide yes)
-			)
-		)
-		(pin "2"
-		)
-		(pin "3"
-		)
-		(pin "1"
-		)
-		(instances
-			(project ""
-				(path "/6cc81634-7f84-4baf-bf6f-e0ba6e6d2a37"
-					(reference "U2")
-					(unit 1)
-				)
-			)
-		)
 	)
 	(symbol
@@
 			)
 		)
-		(property "Footprint" ""
+		(property "Footprint" "Connector_BarrelJack:BarrelJack_CLIFF_FC681465S_SMT_Horizontal"
 			(at 27.94 28.956 0)
 			(effects
@@
 			)
 		)
-		(property "Footprint" ""
+		(property "Footprint" "Potentiometer_THT:Potentiometer_Bourns_3296W_Vertical"
 			(at 34.29 57.15 0)
 			(effects
@@
 			)
 		)
-		(property "Footprint" ""
+		(property "Footprint" "Package_TO_SOT_THT:TO-92"
 			(at 123.19 77.47 0)
 			(effects
@@
 			)
 		)
-		(property "Footprint" ""
+		(property "Footprint" "Package_TO_SOT_THT:TO-92"
 			(at 96.52 101.6 0)
 			(effects
@@
 	)
 	(symbol
+		(lib_id "Connector:Conn_01x03_Pin")
+		(at 63.5 44.45 0)
+		(unit 1)
+		(exclude_from_sim no)
+		(in_bom yes)
+		(on_board yes)
+		(dnp no)
+		(fields_autoplaced yes)
+		(property "Reference" "J2"
+			(at 64.135 36.83 0)
+			(effects
+				(font
+					(size 1.27 1.27)
+				)
+			)
+		)
+		(property "Value" "Conn_01x03_Pin"
+			(at 64.135 39.37 0)
+			(effects
+				(font
+					(size 1.27 1.27)
+				)
+			)
+		)
+		(property "Footprint" "Connector_PinHeader_2.54mm:PinHeader_1x03_P2.54mm_Vertical"
+			(at 63.5 44.45 0)
+			(effects
+				(font
+					(size 1.27 1.27)
+				)
+				(hide yes)
+			)
+		)
+		(property "Datasheet" "~"
+			(at 63.5 44.45 0)
+			(effects
+				(font
+					(size 1.27 1.27)
+				)
+				(hide yes)
+			)
+		)
+		(property "Description" "Generic connector, single row, 01x03, script generated"
+			(at 63.5 44.45 0)
+			(effects
+				(font
+					(size 1.27 1.27)
+				)
+				(hide yes)
+			)
+		)
+		(pin "1"
+		)
+		(pin "2"
+		)
+		(pin "3"
+		)
+		(instances
+			(project ""
+				(path "/6cc81634-7f84-4baf-bf6f-e0ba6e6d2a37"
+					(reference "J2")
+					(unit 1)
+				)
+			)
+		)
+	)
+	(symbol
 		(lib_id "Device:LED")
 		(at 27.94 43.18 0)
@@
 			)
 		)
-		(property "Footprint" ""
+		(property "Footprint" "LED_THT:LED_D5.0mm"
 			(at 27.94 43.18 0)
 			(effects

Commit message: placed all the components
done
Parts:
- removed J1: Barrel_Jack, Connector_BarrelJack:BarrelJack_CLIFF_FC681465S_SMT_Horizontal, symbol Connector:Barrel_Jack
- added C1, C3: C_Polarized_US, symbol Device:C_Polarized_US
- added C2: C_Polarized, symbol Device:C_Polarized
- added D2, D3, D4, D5, D6: 1N4005, Diode_THT:D_DO-41_SOD81_P10.16mm_Horizontal, symbol Diode:1N4005
- added F1: Fuse, symbol Device:Fuse
- added Q3: NPN, Package_TO_SOT_THT:TO-92, symbol Simulation_SPICE:NPN
- added Q4: PNP, Package_TO_SOT_THT:TO-92, symbol Simulation_SPICE:PNP
- added R1, R10, R2, R3, R4, R5, R6, R7, R8, R9: R_US, symbol Device:R_US
- added SW1: SW_SPST, symbol Switch:SW_SPST
- added U2: LM339, symbol Comparator:LM339
- added V1: VSIN, symbol Simulation_SPICE:VSIN
Other:
- moved on the sheet: D1, J2, Q1, Q2, RV1, U1

Commit message: commit wiring done
Connections:
- net at D5.1 (K): now also D3.1 (K), D6.2 (A), R1.1, R2.1
- net at D5.2 (A): now also D4.1 (K), V1.2
- net at R5.1: now also C3.1, Q4.3 (E), R3.1, R4.1, R7.1, R8.1, U1.3 (VO)
- net at R5.2: now also Q2.2 (B), R6.1
- net at R3.2: now also D1.2 (A)
- net at U1.1 (VI): now also C1.1, D6.1 (K)
- net at U1.2 (GND): now also C1.2, C2.2, C3.2, D1.1 (K), D2.2 (A), D4.2 (A), Q1.3 (E), Q3.3 (E), R1.2, R10.2, R6.2, RV1.2, RV1.3
- net at SW1.1 (A): now also V1.1
- net at SW1.2 (B): now also F1.1
- net at RV1.1: now also R8.2, U2.5 (+)
- net at D2.1 (K): now also D3.2 (A), F1.2
- net at Q3.1 (C): now also U2.4 (-)
- net at Q3.2 (B): now also Q1.1 (C), R4.2
- net at R7.2: now also Q2.3 (E)
- net at R2.2: now also Q1.2 (B)
- net at Q2.1 (C): now also C2.1
- net at R9.1: now also U2.2
- net at R9.2: now also Q4.2 (B)
- net at Q4.1 (C): now also R10.1
Other:
- moved on the sheet: C1, C2, C3, D1, Q1, Q2, Q3, Q4, R1, R10, R2, R3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

Commit message: commit
Connections:
- net GNDPWR: now also D4.1 (K), D5.2 (A), V1.2
- net VAC: now also SW1.1 (A), V1.1
Changed lines of the file:
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@@
+	)
+	(junction
+		(at 22.86 106.68)
+		(diameter 0)
+		(color 0 0 0 0)
 	)
 	(junction
@@
 	)
 	(junction
+		(at 22.86 118.11)
+		(diameter 0)
+		(color 0 0 0 0)
+	)
+	(junction
 		(at 69.85 143.51)
 		(diameter 0)
@@
 	(wire
 		(pts
+			(xy 19.05 118.11) (xy 22.86 118.11)
+		)
+		(stroke
+			(width 0)
+			(type default)
+		)
+	)
+	(wire
+		(pts
 			(xy 46.99 132.08) (xy 53.34 132.08)
 		)
@@
 	(wire
 		(pts
+			(xy 22.86 118.11) (xy 29.21 118.11)
+		)
+		(stroke
+			(width 0)
+			(type default)
+		)
+	)
+	(wire
+		(pts
 			(xy 144.78 90.17) (xy 144.78 97.79)
 		)
@@
 	(wire
 		(pts
+			(xy 20.32 106.68) (xy 22.86 106.68)
+		)
+		(stroke
+			(width 0)
+			(type default)
+		)
+	)
+	(wire
+		(pts
 			(xy 41.91 101.6) (xy 41.91 96.52)
 		)
@@
 	(wire
 		(pts
+			(xy 22.86 106.68) (xy 30.48 106.68)
+		)
+		(stroke
+			(width 0)
+			(type default)
+		)
+	)
+	(wire
+		(pts
 			(xy 243.84 121.92) (xy 256.54 121.92)
 		)
@@
 	(wire
 		(pts
+			(xy 22.86 118.11) (xy 22.86 138.43)
+		)
+		(stroke
+			(width 0)
+			(type default)
+		)
+	)
+	(wire
+		(pts
 			(xy 69.85 113.03) (xy 69.85 128.27)
 		)
@@
 	(wire
 		(pts
-			(xy 22.86 116.84) (xy 22.86 138.43)
+			(xy 22.86 116.84) (xy 22.86 118.11)
 		)
 		(stroke
@@
 	(wire
 		(pts
+			(xy 29.21 116.84) (xy 29.21 118.11)
+		)
+		(stroke
+			(width 0)
+			(type default)
+		)
+	)
+	(wire
+		(pts
 			(xy 144.78 113.03) (xy 144.78 128.27)
 		)
@@
 		(pts
 			(xy 91.44 90.17) (xy 92.71 90.17)
+		)
+		(stroke
+			(width 0)
+			(type default)
+		)
+	)
+	(wire
+		(pts
+			(xy 30.48 105.41) (xy 30.48 106.68)
 		)
 		(stroke
@@
 	(symbol
 		(lib_id "power:GNDPWR")
-		(at 50.8 41.91 0)
+		(at 19.05 118.11 270)
 		(unit 1)
 		(exclude_from_sim no)
@@
 		(on_board yes)
 		(dnp no)
-		(fields_autoplaced yes)
 		(property "Reference" "#PWR02"
-			(at 50.8 46.99 0)
+			(at 13.97 118.11 0)
 			(effects
 				(font
@@
 		)
 		(property "Value" "GNDPWR"
-			(at 50.673 45.72 0)
-			(effects
-				(font
-					(size 1.27 1.27)
-				)
+			(at 20.828 115.57 90)
+			(effects
+				(font
+					(size 1.27 1.27)
+				)
+				(justify right)
 			)
 		)
 		(property "Footprint" ""
-			(at 50.8 43.18 0)
+			(at 17.78 118.11 0)
 			(effects
 				(font
@@
 		)
 		(property "Datasheet" ""
-			(at 50.8 43.18 0)
+			(at 17.78 118.11 0)
 			(effects
 				(font
@@
 		)
 		(property "Description" "Power symbol creates a global label with name \"GNDPWR\" , global ground"
-			(at 50.8 41.91 0)
+			(at 19.05 118.11 0)
 			(effects
 				(font
@@
 	(symbol
 		(lib_id "power:PWR_FLAG")
-		(at 45.72 62.23 0)
+		(at 30.48 105.41 0)
 		(unit 1)
 		(exclude_from_sim no)
@@
 		(on_board yes)
 		(dnp no)
-		(fields_autoplaced yes)
 		(property "Reference" "#FLG01"
-			(at 45.72 60.325 0)
+			(at 30.48 103.505 0)
 			(effects
 				(font
@@
 		)
 		(property "Value" "PWR_FLAG"
-			(at 45.72 57.15 0)
+			(at 32.258 100.584 0)
 			(effects
 				(font
@@
 		)
 		(property "Footprint" ""
-			(at 45.72 62.23 0)
+			(at 30.48 105.41 0)
 			(effects
 				(font
@@
 		)
 		(property "Datasheet" "~"
-			(at 45.72 62.23 0)
+			(at 30.48 105.41 0)
 			(effects
 				(font
@@
 		)
 		(property "Description" "Special symbol for telling ERC where power comes from"
-			(at 45.72 62.23 0)
+			(at 30.48 105.41 0)
 			(effects
 				(font
@@
 	(symbol
 		(lib_id "power:VAC")
-		(at 30.48 60.96 0)
+		(at 20.32 106.68 90)
 		(unit 1)
 		(exclude_from_sim no)
@@
 		(on_board yes)
 		(dnp no)
-		(fields_autoplaced yes)
 		(property "Reference" "#PWR03"
-			(at 30.48 63.5 0)
+			(at 22.86 106.68 0)
 			(effects
 				(font
@@
 		)
 		(property "Value" "VAC"
-			(at 30.48 53.34 0)
-			(effects
-				(font
-					(size 1.27 1.27)
-				)
+			(at 18.796 102.87 90)
+			(effects
+				(font
+					(size 1.27 1.27)
+				)
+				(justify left)
 			)
 		)
 		(property "Footprint" ""
-			(at 30.48 60.96 0)
+			(at 20.32 106.68 0)
 			(effects
 				(font
@@
 		)
 		(property "Datasheet" ""
-			(at 30.48 60.96 0)
+			(at 20.32 106.68 0)
 			(effects
 				(font
@@
 		)
 		(property "Description" "Power symbol creates a global label with name \"VAC\""
-			(at 30.48 60.96 0)
+			(at 20.32 106.68 0)
 			(effects
 				(font
@@
 					(unit 1)
 				)
+			)
+		)
+	)
+	(symbol
+		(lib_id "power:PWR_FLAG")
+		(at 29.21 116.84 0)
+		(unit 1)
+		(exclude_from_sim no)
+		(in_bom yes)
+		(on_board yes)
+		(dnp no)
+		(property "Reference" "#FLG02"
+			(at 29.21 114.935 0)
+			(effects
+				(font
+					(size 1.27 1.27)
+				)
+				(hide yes)
+			)
+		)
+		(property "Value" "PWR_FLAG"
+			(at 30.734 111.506 0)
+			(effects
+				(font
+					(size 1.27 1.27)
+				)
+			)
+		)
+		(property "Footprint" ""
+			(at 29.21 116.84 0)
+			(effects
+				(font
+					(size 1.27 1.27)
+				)
+				(hide yes)
+			)
+		)
+		(property "Datasheet" "~"
+			(at 29.21 116.84 0)
+			(effects
+				(font
+					(size 1.27 1.27)
+				)
+				(hide yes)
+			)
+		)
+		(property "Description" "Special symbol for telling ERC where power comes from"
+			(at 29.21 116.84 0)
+			(effects
+				(font
+					(size 1.27 1.27)
+				)
+				(hide yes)
+			)
+		)
+		(pin "1"
+		)
+		(instances
+			(project "PWMGenerator-nkoirala1"
+				(path "/6cc81634-7f84-4baf-bf6f-e0ba6e6d2a37"
+					(reference "#FLG02")
+					(unit 1)
+				)

Commit message: Update PWMGenerator-nkoirala1.kicad_sch
Connections:
- net GNDPWR: now also C1.2, C2.2, C3.2, D1.1 (K), D2.2 (A), D4.2 (A), Q1.3 (E), Q3.3 (E), R1.2, R10.2, R6.2, RV1.2, RV1.3, U1.2 (GND)
- net VCC: now reaches C3.1, Q4.3 (E), R3.1, R4.1, R5.1, R7.1, R8.1, U1.3 (VO)
