File: PWMGenerator-nkoirala1 _B/PWMGenerator-nkoirala1.kicad_sch (KiCad schematic)
At the start: 30 parts, among them J2 Conn_01x03_Pin, Q1 NPN, Q2 PNP, Q3 NPN, Q4 PNP, SW1 SW_SPST, U1 LM7805_TO220, U2 LM339

Commit message: Resistors Footprint
not potentiometer
Parts:
- R1, R10, R2, R3, R4, R5, R6, R7, R8, R9: footprint (none) -> Resistor_SMD:R_0805_2012Metric_Pad1.20x1.40mm_HandSolder
Changed lines of the file:
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@@
 			)
 		)
-		(property "Footprint" ""
+		(property "Footprint" "Resistor_SMD:R_0805_2012Metric_Pad1.20x1.40mm_HandSolder"
 			(at 167.386 101.854 90)
 			(effects
@@
 			)
 		)
-		(property "Footprint" ""
+		(property "Footprint" "Resistor_SMD:R_0805_2012Metric_Pad1.20x1.40mm_HandSolder"
 			(at 133.096 101.854 90)
 			(effects
@@
 			)
 		)
-		(property "Footprint" ""
+		(property "Footprint" "Resistor_SMD:R_0805_2012Metric_Pad1.20x1.40mm_HandSolder"
 			(at 182.626 101.854 90)
 			(effects
@@
 			)
 		)
-		(property "Footprint" ""
+		(property "Footprint" "Resistor_SMD:R_0805_2012Metric_Pad1.20x1.40mm_HandSolder"
 			(at 103.124 127.254 90)
 			(effects
@@
 			)
 		)
-		(property "Footprint" ""
+		(property "Footprint" "Resistor_SMD:R_0805_2012Metric_Pad1.20x1.40mm_HandSolder"
 			(at 227.584 112.014 90)
 			(effects
@@
 			)
 		)
-		(property "Footprint" ""
+		(property "Footprint" "Resistor_SMD:R_0805_2012Metric_Pad1.20x1.40mm_HandSolder"
 			(at 70.866 134.874 90)
 			(effects
@@
 			)
 		)
-		(property "Footprint" ""
+		(property "Footprint" "Resistor_SMD:R_0805_2012Metric_Pad1.20x1.40mm_HandSolder"
 			(at 145.796 101.854 90)
 			(effects
@@
 			)
 		)
-		(property "Footprint" ""
+		(property "Footprint" "Resistor_SMD:R_0805_2012Metric_Pad1.20x1.40mm_HandSolder"
 			(at 197.866 101.854 90)
 			(effects
@@
 			)
 		)
-		(property "Footprint" ""
+		(property "Footprint" "Resistor_SMD:R_0805_2012Metric_Pad1.20x1.40mm_HandSolder"
 			(at 244.856 129.794 90)
 			(effects
@@
 			)
 		)
-		(property "Footprint" ""
+		(property "Footprint" "Resistor_SMD:R_0805_2012Metric_Pad1.20x1.40mm_HandSolder"
 			(at 167.386 129.794 90)
 			(effects

Commit message: Capacity FootPrint
Parts:
- C2: footprint (none) -> Capacitor_SMD:C_0805_2012Metric
Changed lines of the file:
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@@
 			)
 		)
-		(property "Footprint" ""
+		(property "Footprint" "Capacitor_SMD:C_0805_2012Metric"
 			(at 182.5752 133.35 0)
 			(effects

Commit message: Diode
Including LED Done
Parts:
- D1: value LED -> GREEN
- D2, D3, D4, D5, D6: value 1N4005 -> 1N4005G; footprint Diode_THT:D_DO-41_SOD81_P10.16mm_Horizontal -> Diode_SMD:D_0805_2012Metric_Pad1.15x1.40mm_HandSolder
Changed lines of the file:
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@@
 			)
 		)
-		(property "Value" "1N4005"
+		(property "Value" "1N4005G"
 			(at 55.88 123.1899 90)
 			(effects
@@
 			)
 		)
-		(property "Footprint" "Diode_THT:D_DO-41_SOD81_P10.16mm_Horizontal"
+		(property "Footprint" "Diode_SMD:D_0805_2012Metric_Pad1.15x1.40mm_HandSolder"
 			(at 48.895 121.92 0)
 			(effects
@@
 			)
 		)
-		(property "Value" "1N4005"
+		(property "Value" "1N4005G"
 			(at 44.45 123.1899 90)
 			(effects
@@
 			)
 		)
-		(property "Footprint" "Diode_THT:D_DO-41_SOD81_P10.16mm_Horizontal"
+		(property "Footprint" "Diode_SMD:D_0805_2012Metric_Pad1.15x1.40mm_HandSolder"
 			(at 46.355 121.92 0)
 			(effects
@@
 			)
 		)
-		(property "Value" "1N4005"
+		(property "Value" "1N4005G"
 			(at 44.45 106.6799 90)
 			(effects
@@
 			)
 		)
-		(property "Footprint" "Diode_THT:D_DO-41_SOD81_P10.16mm_Horizontal"
+		(property "Footprint" "Diode_SMD:D_0805_2012Metric_Pad1.15x1.40mm_HandSolder"
 			(at 37.465 105.41 0)
 			(effects
@@
 			)
 		)
-		(property "Value" "1N4005"
+		(property "Value" "1N4005G"
 			(at 73.66 86.36 0)
 			(effects
@@
 			)
 		)
-		(property "Footprint" "Diode_THT:D_DO-41_SOD81_P10.16mm_Horizontal"
+		(property "Footprint" "Diode_SMD:D_0805_2012Metric_Pad1.15x1.40mm_HandSolder"
 			(at 73.66 85.725 0)
 			(effects
@@
 			)
 		)
-		(property "Value" "1N4005"
+		(property "Value" "1N4005G"
 			(at 55.88 106.6799 90)
 			(effects
@@
 			)
 		)
-		(property "Footprint" "Diode_THT:D_DO-41_SOD81_P10.16mm_Horizontal"
+		(property "Footprint" "Diode_SMD:D_0805_2012Metric_Pad1.15x1.40mm_HandSolder"
 			(at 57.785 105.41 0)
 			(effects
@@
 			)
 		)
-		(property "Value" "LED"
+		(property "Value" "GREEN"
 			(at 135.89 132.3974 90)
 			(effects

Commit message: 2N3904 And 2n3906
Footprint
Parts:
- Q1, Q3: value NPN -> 2N3904; footprint Package_TO_SOT_THT:TO-92 -> Package_TO_SOT_SMD:SOT-23
- Q2, Q4: value PNP -> 2N3906; footprint Package_TO_SOT_THT:TO-92 -> Package_TO_SOT_SMD:SOT-23
Changed lines of the file:
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@@
 			)
 		)
-		(property "Value" "NPN"
+		(property "Value" "2N3904"
 			(at 156.21 129.5399 0)
 			(effects
@@
 			)
 		)
-		(property "Footprint" "Package_TO_SOT_THT:TO-92"
+		(property "Footprint" "Package_TO_SOT_SMD:SOT-23"
 			(at 214.63 128.27 0)
 			(effects
@@
 			)
 		)
-		(property "Value" "NPN"
+		(property "Value" "2N3904"
 			(at 124.46 129.5399 0)
 			(effects
@@
 			)
 		)
-		(property "Footprint" "Package_TO_SOT_THT:TO-92"
+		(property "Footprint" "Package_TO_SOT_SMD:SOT-23"
 			(at 182.88 128.27 0)
 			(effects
@@
 			)
 		)
-		(property "Value" "PNP"
+		(property "Value" "2N3906"
 			(at 184.15 116.8399 0)
 			(effects
@@
 			)
 		)
-		(property "Footprint" "Package_TO_SOT_THT:TO-92"
+		(property "Footprint" "Package_TO_SOT_SMD:SOT-23"
 			(at 214.63 115.57 0)
 			(effects
@@
 			)
 		)
-		(property "Value" "PNP"
+		(property "Value" "2N3906"
 			(at 246.38 114.2999 0)
 			(effects
@@
 			)
 		)
-		(property "Footprint" "Package_TO_SOT_THT:TO-92"
+		(property "Footprint" "Package_TO_SOT_SMD:SOT-23"
 			(at 276.86 113.03 0)
 			(effects

Commit message: Commit
Fuse but its wrong need to do it
Parts:
- removed F1: Fuse, symbol Device:Fuse
- added F2: Polyfuse, Fuse:Fuse_1206_3216Metric, symbol Device:Polyfuse
- U2: footprint (none) -> Package_SO:SOIC-14-16_3.9x9.9mm_P1.27mm
Connections:
- net at SW1.2 (B): now also F2.1
- net at D2.1 (K), D3.2 (A): now also F2.2
Changed lines of the file:
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@@
+	)
+	(symbol
+		(lib_id "Device:Polyfuse")
+		(at 35.56 88.9 90)
+		(unit 1)
+		(exclude_from_sim no)
+		(in_bom yes)
+		(on_board yes)
+		(dnp no)
+		(property "Reference" "F2"
+			(at 34.798 85.852 90)
+			(effects
+				(font
+					(size 1.27 1.27)
+				)
+			)
+		)
+		(property "Value" "Polyfuse"
+			(at 35.56 85.852 90)
+			(effects
+				(font
+					(size 1.27 1.27)
+				)
+				(hide yes)
+			)
+		)
+		(property "Footprint" "Fuse:Fuse_1206_3216Metric"
+			(at 40.64 87.63 0)
+			(effects
+				(font
+					(size 1.27 1.27)
+				)
+				(justify left)
+				(hide yes)
+			)
+		)
+		(property "Datasheet" "~"
+			(at 35.56 88.9 0)
+			(effects
+				(font
+					(size 1.27 1.27)
+				)
+				(hide yes)
+			)
+		)
+		(property "Description" "Resettable fuse, polymeric positive temperature coefficient"
+			(at 35.56 88.9 0)
+			(effects
+				(font
+					(size 1.27 1.27)
+				)
+				(hide yes)
+			)
+		)
+		(pin "1"
+		)
+		(pin "2"
+		)
+		(instances
+			(project ""
+				(path "/6cc81634-7f84-4baf-bf6f-e0ba6e6d2a37"
+					(reference "F2")
+					(unit 1)
+				)
+			)
+		)
 	)
 	(symbol
@@
 		(dnp no)
 		(property "Reference" "J2"
-			(at 260.35 97.536 0)
+			(at 261.874 97.536 0)
 			(effects
 				(font
@@
 			)
 		)
-		(property "Footprint" ""
+		(property "Footprint" "Package_SO:SOIC-14-16_3.9x9.9mm_P1.27mm"
 			(at 210.82 110.49 0)
 			(effects
@@
 					(unit 1)
 				)
-			)
-		)
-	)
-	(symbol
-		(lib_id "Device:Fuse")
-		(at 35.56 88.9 90)
-		(unit 1)
-		(exclude_from_sim no)
-		(in_bom yes)
-		(on_board yes)
-		(dnp no)
-		(property "Reference" "F1"
-			(at 35.814 86.36 90)
-			(effects
-				(font
-					(size 1.27 1.27)
-				)
-			)
-		)
-		(property "Value" "Fuse"
-			(at 35.56 85.09 90)
-			(effects
-				(font
-					(size 1.27 1.27)
-				)
-				(hide yes)
-			)
-		)
-		(property "Footprint" ""
-			(at 35.56 90.678 90)
-			(effects
-				(font
-					(size 1.27 1.27)
-				)
-				(hide yes)
-			)
-		)
-		(property "Datasheet" "~"
-			(at 35.56 88.9 0)
-			(effects
-				(font
-					(size 1.27 1.27)
-				)
-				(hide yes)
-			)
-		)
-		(property "Description" "Fuse"
-			(at 35.56 88.9 0)
-			(effects
-				(font
-					(size 1.27 1.27)
-				)
-				(hide yes)
-			)
-		)
-		(pin "1"
-		)
-		(pin "2"
-		)
-		(instances
-			(project ""
-				(path "/6cc81634-7f84-4baf-bf6f-e0ba6e6d2a37"
-					(reference "F1")
-					(unit 1)
-				)
