File: PWMGenerator-nkoirala1 _C/PWMGenerator-nkoirala1.kicad_sch (KiCad schematic)
At the start: 30 parts, among them J2 Conn_01x03_Pin, Q2 2N3906, Q4 2N3904, Q5 2N3906, Q6 2N3904, SW1 SW_SPST, U1 LM7805_TO220, U2 LM339

Commit message: commit
fixing some isses
Parts:
- removed U2: LM339, Package_SO:SOIC-14-16_3.9x9.9mm_P1.27mm, symbol Comparator:LM339
- added U3: LM339, Package_SO:SOIC-14-16_3.9x9.9mm_P1.27mm, symbol Comparator:LM339
Connections:
- net GND: now also U3.12 (V-)
- net VCC: now also U3.3 (V+)
- net at R8.2, RV1.1: now also U3.5 (+)
- net at C2.1, Q2.1 (C), Q6.3 (C): now also U3.4 (-)
- net at R9.1: now also U3.2

Commit message: had my footprint wrong fr lm339
Updated
Parts:
- U3: footprint Package_SO:SOIC-14-16_3.9x9.9mm_P1.27mm -> Package_SO:SOIC-14_3.9x8.7mm_P1.27mm
Changed lines of the file:
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@@
 			)
 		)
-		(property "Footprint" "Package_SO:SOIC-14-16_3.9x9.9mm_P1.27mm"
+		(property "Footprint" "Package_SO:SOIC-14_3.9x8.7mm_P1.27mm"
 			(at 210.82 104.14 0)
 			(effects
@@
 			)
 		)
-		(property "Footprint" "Package_SO:SOIC-14-16_3.9x9.9mm_P1.27mm"
+		(property "Footprint" "Package_SO:SOIC-14_3.9x8.7mm_P1.27mm"
 			(at 227.33 31.75 0)
 			(effects
@@
 			)
 		)
-		(property "Footprint" "Package_SO:SOIC-14-16_3.9x9.9mm_P1.27mm"
+		(property "Footprint" "Package_SO:SOIC-14_3.9x8.7mm_P1.27mm"
 			(at 210.82 104.14 0)
 			(effects
@@
 			)
 		)
-		(property "Footprint" "Package_SO:SOIC-14-16_3.9x9.9mm_P1.27mm"
+		(property "Footprint" "Package_SO:SOIC-14_3.9x8.7mm_P1.27mm"
 			(at 228.6 63.5 0)
 			(effects
@@
 			)
 		)
-		(property "Footprint" "Package_SO:SOIC-14-16_3.9x9.9mm_P1.27mm"
+		(property "Footprint" "Package_SO:SOIC-14_3.9x8.7mm_P1.27mm"
 			(at 228.6 46.99 0)
 			(effects
